File: pc-xt-256-640k/pc-xt-256-640k.kicad_sch (KiCad schematic)
At the start: 0 parts

Commit message: add two first two empty schematic pages
Other:
- added sheet Processor and Support (processor-and-support.kicad_sch)
- added sheet Wait State Generator (wait-state-generator.kicad_sch)
Changed lines of the file:
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@@
 		(rev "MAR86")
+	)
+	(sheet
+		(at 25.4 50.8)
+		(size 38.1 12.7)
+		(exclude_from_sim no)
+		(in_bom yes)
+		(on_board yes)
+		(dnp no)
+		(fields_autoplaced yes)
+		(stroke
+			(width 0.1524)
+			(type solid)
+		)
+		(fill
+			(color 0 0 0 0.0000)
+		)
+		(property "Sheetname" "Wait State Generator"
+			(at 25.4 50.0884 0)
+			(effects
+				(font
+					(size 1.27 1.27)
+				)
+				(justify left bottom)
+			)
+		)
+		(property "Sheetfile" "wait-state-generator.kicad_sch"
+			(at 25.4 64.0846 0)
+			(effects
+				(font
+					(size 1.27 1.27)
+				)
+				(justify left top)
+			)
+		)
+		(instances
+			(project "pc-xt-256-640k"
+				(path "/943bb5a2-da39-4fff-b96b-04b08b617828"
+					(page "3")
+				)
+			)
+		)
+	)
+	(sheet
+		(at 25.4 25.4)
+		(size 38.1 12.7)
+		(exclude_from_sim no)
+		(in_bom yes)
+		(on_board yes)
+		(dnp no)
+		(fields_autoplaced yes)
+		(stroke
+			(width 0.1524)
+			(type solid)
+		)
+		(fill
+			(color 0 0 0 0.0000)
+		)
+		(property "Sheetname" "Processor and Support"
+			(at 25.4 24.6884 0)
+			(effects
+				(font
+					(size 1.27 1.27)
+				)
+				(justify left bottom)
+			)
+		)
+		(property "Sheetfile" "processor-and-support.kicad_sch"
+			(at 25.4 38.6846 0)
+			(effects
+				(font
+					(size 1.27 1.27)
+				)
+				(justify left top)
+			)
+		)
+		(instances
+			(project "pc-xt-256-640k"
+				(path "/943bb5a2-da39-4fff-b96b-04b08b617828"
+					(page "2")
+				)
+			)
+		)
 	)
 	(sheet_instances
