File: pc-xt-256-640k/processor-and-support.kicad_sch (KiCad schematic)
At the start: 0 parts

Commit message: Started sheet 1 schematic
Parts:
- added C1: 5-30PF, symbol Device:C_Variable
- added R1, R2: 510, symbol Device:R_US
- added RN1-1: 4.7K, symbol Device:R_US
- added U1: 8284A, Package_DIP:DIP-18_W7.62mm, symbol ibm_intel:8284A
- added U1: LS373, symbol ibm_74xx:LS373
- added U2: LS245, symbol ibm_74xx:LS245
- added U22: LS04, symbol ibm_74xx:LS04
- added U3: 8087, Package_DIP:DIP-40_W15.24mm, symbol ibm_intel:8087
- added U4: 8088, Package_DIP:DIP-40_W15.24mm, symbol ibm_intel:8088
- added Y1: 14.31818MHZ, symbol Device:Crystal
Connections:
- new net: C1.2, R1.1, U1.17 (X1)
- new net: C1.1, Y1.2
- new net: U1.13 (F/~{C}), U22.10
- new net: R2.1, U1.16 (X2), Y1.1
- new net: RN1-1.2, U22.11
- new net AA10: U4.6 (A10)
- new net AA11: U4.5 (A11)
- new net AA12: U4.4 (A12)
- new net AA13: U4.3 (A13)
- new net AA14: U4.2 (A14)
- new net AA15: U4.39 (A15)
- new net AA16: U4.38 (A16)
- new net AA17: U4.37 (A17)
- new net AA18: U4.36 (A18)
- new net AA19: U4.35 (A19)
- new net AA8: U4.8 (A8)
- new net AA9: U4.7 (A9)
- new net AD0: U1.18 (D), U2.9 (A8), U3.16 (AD0), U4.16 (AD0)
- new net AD1: U1.17 (D), U2.8 (A7), U3.15 (AD1), U4.15 (AD1)
- new net AD2: U1.14 (D), U2.7 (A6), U3.14 (AD2), U4.14 (AD2)
- new net AD3: U1.13 (D), U2.6 (A5), U3.13 (AD3), U4.13 (AD3)
- new net AD4: U1.8 (D), U2.5 (A4), U3.12 (AD4), U4.12 (AD4)
- new net AD5: U1.7 (D), U2.4 (A3), U3.11 (AD5), U4.11 (AD5)
- new net AD6: U1.4 (D), U2.3 (A2), U3.10 (AD6), U4.10 (AD6)
- new net AD7: U1.3 (D), U2.2 (A1), U3.9 (AD7), U4.9 (AD7)
- new net CLK88: U1.8 (CLK), U3.19 (CLK), U4.19 (CLK)
- new net Earth: R1.2, R2.2, U1.1 (CSYNC), U1.15 (~{ASYNC})
- new net LOCK: U4.29 (LOCK)
- new net NMI: U4.17 (NMI)
- new net READY: U1.5 (RDY), U3.22 (READY), U4.22 (READY)
- new net RESET: U1.10 (RES), U3.21 (RESET), U4.21 (RESET)
- new net ~{S0}: U4.26 (~{S0})
- new net ~{S1}: U4.27 (~{S1})
- new net ~{S2}: U4.28 (~{S2})
